Commit message: Sync scenario naming/algorithm set and fix LiDAR/payload self-collision
Renamed the A-E scenario scheme to the current 1_ideal /
2_unmapped_{persistent,transient} matrix everywhere (README, launch
files, scenario_spawner_node), matching docs/experiment_protocol.md in
the Jetson repo. Also documents DQN -> CQL/SARSA in prose.

scenario_spawner_node gains the transient variant's own-timer obstacle
removal (mirrors sim2d/room_env.py's _maybe_clear_transient_obstacles).

Unrelated fixes picked up in the same pass:
- deck_z raised from 0.105 to 0.175 m: at the old height the payload
  plate/tank/mast base self-intersected the LiDAR's scan ring, latching
  a permanent ~0.13 m "obstacle" reading and the emergency stop with it.
- Gazebo camera plugin remapping was publishing under `~/image_raw`
  instead of `front/image_raw`, which camera_stream_node's source
  override never actually matched.

Co-Authored-By: Claude Sonnet 5 <noreply@anthropic.com>
Claude-Session: https://claude.ai/code/session_013ugFJhFKiecRyM3nr8CtvK

File: src/myagv_sprayer_description/urdf/common_properties.xacro (robot description, xacro)
@@ -18,5 +18,10 @@
   <xacro:property name="camera_z"     value="0.060"/>
   <!-- payload -->
-  <xacro:property name="deck_z"       value="0.105"/>   <!-- top surface of chassis -->
+  <!-- Raised on standoffs above the LiDAR (lidar_z=0.135, cylinder half-height 0.02,
+       so its scan plane top is 0.155): the payload plate, tank and mast base all sit
+       here, and without this margin they self-intersect the LiDAR's 360 deg scan ring,
+       permanently reading a ~0.13 m "obstacle" and latching the emergency stop. mast_top_z,
+       nozzle_z and camera_z are absolute heights and are unaffected by this offset. -->
+  <xacro:property name="deck_z"       value="0.175"/>
   <xacro:property name="tank_radius"  value="0.055"/>
   <xacro:property name="tank_height"  value="0.140"/>   <!-- ~1 L -->

File: src/myagv_sprayer_description/urdf/sensors.gazebo.xacro (robot description, xacro)
@@ -64,6 +64,6 @@
         <ros>
           <namespace>camera</namespace>
-          <remapping>~/image_raw:=image_raw</remapping>
-          <remapping>~/camera_info:=camera_info</remapping>
+          <remapping>front/image_raw:=image_raw</remapping>
+          <remapping>front/camera_info:=camera_info</remapping>
         </ros>
         <camera_name>front</camera_name>
