Commit message: Commit the three-marker world and the missing collision geometry
Both were sitting in the working tree only. The world HEAD carried had 4 ArUco
stands, one per tray; the tree has 12, three per tray sharing the tray's id.
That design is what makes a marker-only goal workable at all -- cv2.aruco decodes
within ~20-25 deg of a marker's normal, so a single dock-face marker left each
tray unreadable from most approach directions, and myagv_sprayer_jetson's arrival
test now depends on a sighting from any side. A fresh checkout of this repo would
therefore have failed tools/check_layout.py against the Jetson side.

The URDF gains collision geometry for parts that were visual-only: the bumper
strip (Gazebo's front face stopped at 0.155 while the real one is at 0.165), the
mast, and the nozzle, which reaches 5 cm further forward than the bumper. All
sit clear of the LiDAR's 0.135 m scan plane, so none of them changes what the
scan sees -- they change what can collide.

check_layout.py agrees across all three repos on this state (36 checks).

Co-Authored-By: Claude Opus 5 <noreply@anthropic.com>

File: src/myagv_sprayer_description/urdf/myagv_base.xacro (robot description, xacro)
@@ -50,4 +50,11 @@
         <geometry><box size="${base_length} ${base_width} ${base_height}"/></geometry>
       </collision>
+      <!-- The bumper strip was visual-only, so Gazebo's front face stopped at
+           0.155 while the real robot's is at 0.165. Both sit well below the
+           LiDAR's 0.135 m scan plane, so neither shows up in the scan. -->
+      <collision>
+        <origin xyz="${base_length/2 + 0.005} 0 0.03" rpy="0 0 0"/>
+        <geometry><box size="0.01 ${base_width} 0.03"/></geometry>
+      </collision>
       <inertial>
         <origin xyz="0 0 0.05" rpy="0 0 0"/>
@@ -85,4 +92,10 @@
         <material name="agv_dark"/>
       </visual>
+      <!-- x reaches 0.160, inside the bumper's 0.165, so this adds nothing to the
+           floor-plane footprint. It is however the highest solid on the robot
+           (z = 0.46), so it is the one that decides clearance under an overhang. -->
+      <collision>
+        <geometry><box size="0.02 0.06 0.02"/></geometry>
+      </collision>
       <inertial>
         <mass value="0.03"/>

File: src/myagv_sprayer_description/urdf/sprayer_payload.xacro (robot description, xacro)
@@ -72,4 +72,7 @@
         <material name="agv_dark"/>
       </visual>
+      <collision>
+        <geometry><box size="0.045 0.020 0.015"/></geometry>
+      </collision>
       <inertial>
         <mass value="0.01"/>
@@ -92,4 +95,11 @@
         <material name="agv_grey"/>
       </visual>
+      <!-- The mast spans z = 0.175..0.46, so it overlaps a seedling tray's 0.25 m
+           collision box. It sits at x = 0.140 though, behind the front bumper's
+           0.165, so the bumper always makes contact first. -->
+      <collision>
+        <origin xyz="0 0 ${(mast_top_z - deck_z)/2}" rpy="0 0 0"/>
+        <geometry><cylinder radius="0.006" length="${mast_top_z - deck_z}"/></geometry>
+      </collision>
       <inertial>
         <mass value="0.05"/>
@@ -109,4 +119,13 @@
         <material name="nozzle_teal"/>
       </visual>
+      <!-- Reaches x = 0.2145, i.e. 5 cm further forward than the bumper, at
+           z = 0.38. Above every prop in the room (tallest is the bucket at 0.28)
+           but well under the 2.5 m walls, so this is the link that decides a
+           nose-first wall contact. Gazebo resolves that in 3D for free; sim2d
+           needs the explicit height tiers in layout.ROBOT_FOOTPRINT_HIGH. -->
+      <collision>
+        <origin xyz="0.012 0 0" rpy="0 ${pi/2} 0"/>
+        <geometry><cylinder radius="0.008" length="0.025"/></geometry>
+      </collision>
       <inertial>
         <mass value="0.02"/>
